File: PCB/Xiao Arrow Pad.kicad_pcb (KiCad board)
At the start: 2 copper layers, 78.7 x 46.7 mm, 12 parts, among them SW1 SW_Push, SW2 SW_Push, SW3 SW_Push, SW4 SW_Push, SW5 SW_Push, U1 XIAO-RP2040-DIP

Commit message: Changes
Parts:
- removed the REF** at (178.3, 99.1)
- removed the REF** at (104.6, 99.0)
- removed the REF** at (178.3, 140.7)
- removed the REF** at (104.6, 140.7)
- added REF**: MountingHole_2.2mm_M2, MountingHole:MountingHole_2.2mm_M2, F.Cu at (178.3, 99.1)
- added REF**: MountingHole_2.2mm_M2, MountingHole:MountingHole_2.2mm_M2, F.Cu at (104.7, 140.7)
- added REF**: MountingHole_2.2mm_M2, MountingHole:MountingHole_2.2mm_M2, F.Cu at (104.7, 99.1)
- added REF**: MountingHole_2.2mm_M2, MountingHole:MountingHole_2.2mm_M2, F.Cu at (178.2, 140.7)
Connections:
- D1 pad 2: (no net) -> Net-(D1-DOUT)
- D2 pad 2: (no net) -> unconnected-(D2-DOUT-Pad2)
Routing:
- net Net-(D1-DOUT): track 0.00 -> 65.3 mm

Commit message: Changes
Routing:
- net Net-(D1-DOUT): track 65.3 -> 75.6 mm, vias 0 -> 4
